File: pcb/pcb.sch (KiCad schematic (older format))
At the start: 19 parts, among them P1 Power, P2 Analog, P3 Digital, P4 Digital, P5 CONN_01X01, P6 CONN_01X01, P7 CONN_01X01, P8 CONN_01X01, Q1 TIP120

Commit message: fix sch and pcb bug: diode connect to magnet now
Connections:
- wire segments 61 -> 62
Changed lines of the file:
@@
 $EndComp
-Wire Wire Line
-	6300 2300 6300 3300
 Wire Wire Line
 	2750 2550 2750 3400
@@
 Wire Wire Line
 	5650 2200 6300 2200
-Wire Wire Line
-	5650 3000 5650 3400
 $Comp
 L power:GND #PWR0101
@@
 F 3 "" H 5050 3400 50  0000 C CNN
 	1    5050 3400
-	1    0    0    -1
-$EndComp
-$Comp
-L power:GND #PWR0104
-U 1 1 5C2A2262
-P 5650 3400
-F 0 "#PWR0104" H 5650 3150 50  0001 C CNN
-F 1 "GND" H 5650 3250 50  0000 C CNN
-F 2 "" H 5650 3400 50  0000 C CNN
-F 3 "" H 5650 3400 50  0000 C CNN
-	1    5650 3400
 	1    0    0    -1
 $EndComp
@@
 Text Label 4300 4800 0    50   ~ 0
 A4(SDA)
+Wire Wire Line
+	5650 3000 6300 3000
+Wire Wire Line
+	6300 2300 6300 3000
+Connection ~ 6300 3000
+Wire Wire Line
+	6300 3000 6300 3300
 $EndSCHEMATC
